File: KiCad/MZ80k_SD/MZ80k_SD.kicad_pcb (KiCad board)
At the start: 2 copper layers, 100 x 100 mm, 18 parts, among them J1 MZ-80K BUS, J2 Micro_SD_Card_Kit, J3 INT VCC, J4 EXT 5V, U1 GAL22V10, U2 28C64, U3 8255, U4 Arduino_Pro_Mini_5V

Commit message: Add files via upload
Other:
- board text added: "0.1uF"
- board text added: "10uF"
- board text added: "28C64"
- board text added: "8255"
- board text added: "Arduino Pro Mini 5V"
- board text added: "EXT 5V"
- board text added: "GAL22V10"
- board text added: "INT VCC"
- board text added: "INT/EXT"
- board text added: "MZ-80K BUS"
- board text added: "SD/CMT"

Commit message: Add files via upload
Connections:
- U2 pad 1: (no net) -> +5V
Routing:
- net +5V: track 195.9 -> 202.3 mm
Other:
- board text added: "MZ-80K SD-CARD UNIT Rev1.2"
- board text removed: "MZ-80K SD-CARD UNIT Rev1.1"

Commit message: Add files via upload
Parts:
- added C4: 0.1uF, Capacitor_THT:C_Rect_L4.0mm_W2.5mm_P2.50mm, F.Cu at (127.6, 107.3)
- added C5: 0.1uF, Capacitor_THT:C_Rect_L4.0mm_W2.5mm_P2.50mm, F.Cu at (127.6, 139.1)
- added U5: 74LS30, Package_DIP:DIP-14_W7.62mm_LongPads, F.Cu at (123.8, 104.8)
- added U6: 74LS30, Package_DIP:DIP-14_W7.62mm_LongPads, F.Cu at (123.8, 136.5)
- C6: renamed from C4; value 10uF -> 100uF
- U1: value GAL22V10 -> 74LS04; footprint Package_DIP:DIP-24_W7.62mm_LongPads -> Package_DIP:DIP-14_W7.62mm_LongPads
- U2: value 28C64 -> 2764
- moved U1 43.2 mm to (123.8, 120.7)
- moved C1 40.8 mm to (127.6, 123.2), turned to 270 degrees
- moved C2 23.6 mm to (142.2, 90.2)
- moved U2 23.6 mm to (138.4, 80.9)
- moved C3 21.4 mm to (131.4, 138.4)
- moved U3 21.0 mm to (183.5, 128.9)
- moved U4 3.42 mm to (175.3, 107.3)
- moved C6 3.17 mm to (133.3, 64.8)
- moved J2 1.91 mm to (174.6, 86.4)
Connections:
- C1 pad 1: +5V -> GND
- C1 pad 2: GND -> +5V
- J1 pad 10: (no net) -> GND
- J1 pad 14: (no net) -> GND
- J1 pad 18: (no net) -> GND
- J1 pad 26: (no net) -> GND
- J1 pad 36: (no net) -> GND
- J1 pad 38: (no net) -> GND
- J1 pad 40: (no net) -> GND
- J1 pad 42: (no net) -> GND
- J1 pad 44: (no net) -> GND
- J1 pad 46: (no net) -> GND
- J1 pad 48: (no net) -> GND
- J1 pad 50: (no net) -> GND
- J1 pad 6: (no net) -> GND
- U1 pad 1: Net-(J1-Pad1) -> Net-(J1-Pad8)
- U1 pad 10: Net-(J1-Pad27) -> Net-(U1-Pad10)
- U1 pad 11: (no net) -> Net-(J1-Pad21)
- U1 pad 12: GND -> Net-(U1-Pad12)
- U1 pad 13: Net-(J1-Pad8) -> Net-(J1-Pad12)
- U1 pad 14: Net-(J1-Pad12) -> +5V
- U1 pad 2: Net-(J1-Pad3) -> Net-(U1-Pad2)
- U1 pad 3: Net-(J1-Pad5) -> GND
- U1 pad 4: Net-(J1-Pad7) -> (no net)
- U1 pad 5: Net-(J1-Pad17) -> GND
- U1 pad 6: Net-(J1-Pad19) -> (no net)
- U1 pad 7: Net-(J1-Pad21) -> GND
- U1 pad 8: Net-(J1-Pad23) -> Net-(U1-Pad8)
- U1 pad 9: Net-(J1-Pad25) -> Net-(J1-Pad27)
- U2 pad 20: Net-(U1-Pad23) -> Net-(U2-Pad20)
- U2 pad 22: Net-(U1-Pad19) -> Net-(J1-Pad16)
- U3 pad 36: Net-(U1-Pad17) -> Net-(J1-Pad20)
- U3 pad 5: Net-(U1-Pad18) -> Net-(J1-Pad16)
- U3 pad 6: Net-(U1-Pad22) -> Net-(U3-Pad6)
Routing:
- net Net-(J1-Pad45): track 91.8 -> 202.3 mm, vias 0 -> 1
- net Net-(J1-Pad35): track 57.1 -> 158.5 mm, vias 1 -> 2
- net Net-(J1-Pad20): track 30.6 -> 128.9 mm, vias 0 -> 1
- net Net-(U3-Pad6): track 0.00 -> 91.3 mm
- net Net-(J1-Pad16): track 25.0 -> 115.5 mm, vias 0 -> 1
- net Net-(J1-Pad39): track 59.5 -> 142.7 mm, vias 1 -> 3
- net Net-(J1-Pad31): track 65.3 -> 146.6 mm
- net Net-(U1-Pad17): track 74.2 -> 0.00 mm, vias 2 -> 0
- net Net-(U1-Pad18): track 62.6 -> 0.00 mm, vias 3 -> 0
- net Net-(J1-Pad29): track 67.1 -> 128.0 mm, vias 1 -> 2
- net Net-(U1-Pad22): track 60.5 -> 0.00 mm, vias 2 -> 0
- net GND: track 297.1 -> 353.3 mm
- net Net-(J1-Pad43): track 67.5 -> 122.7 mm, vias 0 -> 3
- net Net-(J1-Pad41): track 65.5 -> 116.2 mm
- net Net-(U1-Pad23): track 43.5 -> 0.00 mm, vias 1 -> 0
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Other:
- board text added: "100uF"
- board text added: "2764"
- board text added: "74LS04"
- board text added: "74LS30"
- board text added: "MZ-80K SD-CARD UNIT Rev1.5.1"
- board text removed: "10uF"
- board text removed: "28C64"
- board text removed: "GAL22V10"
- board text removed: "MZ-80K SD-CARD UNIT Rev1.2"

Commit message: Add files via upload
Connections:
- U1 pad 5: GND -> Net-(J1-Pad32)
- U1 pad 6: (no net) -> Net-(U1-Pad6)
- U4 pad 3: (no net) -> Net-(U1-Pad6)
Routing:
- net Net-(U1-Pad6): track 0.00 -> 67.8 mm, vias 0 -> 1
- net Net-(J1-Pad35): track 158.5 -> 110.3 mm, vias 2 -> 1
- net Net-(J1-Pad47): track 142.0 -> 178.9 mm, vias 2 -> 1
- net Net-(J1-Pad45): track 202.3 -> 168.6 mm
- net Net-(J1-Pad39): track 142.7 -> 111.9 mm, vias 3 -> 1
- net Net-(J1-Pad31): track 146.6 -> 118.2 mm
- net Net-(J1-Pad21): track 93.8 -> 75.6 mm, vias 0 -> 1
- net Net-(J1-Pad32): track 108.7 -> 92.9 mm, vias 0 -> 2
- net Net-(J2-Pad5): track 40.8 -> 55.2 mm
- net Net-(U3-Pad6): track 91.3 -> 77.2 mm
- net Net-(J1-Pad5): track 38.2 -> 50.4 mm, vias 1 -> 0
- net Net-(J1-Pad3): track 43.0 -> 54.0 mm, vias 1 -> 0
- net Net-(U2-Pad20): track 31.3 -> 21.3 mm
- net Net-(J1-Pad43): track 122.7 -> 113.6 mm, vias 3 -> 1
- net Net-(J1-Pad27): track 70.0 -> 79.1 mm
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Other:
- board text added: "MZ-80K SD-CARD UNIT Rev1.5.2"
- board text removed: "MZ-80K SD-CARD UNIT Rev1.5.1"
