File: KiCad/MZ80k_SD/MZ80k_SD.kicad_pcb (KiCad board)
At the start: 2 copper layers, 100 x 100 mm, 22 parts, among them J1 MZ-80K BUS, J2 Micro_SD_Card_Kit, J3 INT VCC, J4 EXT 5V, U1 74LS04, U2 2764, U3 8255, U4 Arduino_Pro_Mini_5V, U5 74LS30, U6 74LS30

Commit message: Add files via upload
Connections:
- net Net-(J1-Pad1) renamed /A15
- net Net-(J1-Pad11) renamed /A10
- net Net-(J1-Pad12) renamed /~IORQ
- net Net-(J1-Pad13) renamed /A9
- net Net-(J1-Pad15) renamed /A8
- net Net-(J1-Pad16) renamed /~RD
- net Net-(J1-Pad17) renamed /A7
- net Net-(J1-Pad19) renamed /A6
- net Net-(J1-Pad20) renamed /~WR
- net Net-(J1-Pad21) renamed /A5
- net Net-(J1-Pad23) renamed /A4
- net Net-(J1-Pad25) renamed /A3
- net Net-(J1-Pad27) renamed /A2
- net Net-(J1-Pad29) renamed /A1
- net Net-(J1-Pad3) renamed /A14
- net Net-(J1-Pad31) renamed /A0
- net Net-(J1-Pad32) renamed /RESET
- net Net-(J1-Pad35) renamed /D7
- net Net-(J1-Pad37) renamed /D6
- net Net-(J1-Pad39) renamed /D5
- net Net-(J1-Pad41) renamed /D4
- net Net-(J1-Pad43) renamed /D3
- net Net-(J1-Pad45) renamed /D2
- net Net-(J1-Pad47) renamed /D1
- net Net-(J1-Pad49) renamed /D0
- net Net-(J1-Pad5) renamed /A13
- net Net-(J1-Pad7) renamed /A12
- net Net-(J1-Pad8) renamed /~MREQ
- net Net-(J1-Pad9) renamed /A11

Commit message: Add files via upload
Parts:
- added J5: MicroSD Card Adapter, Connector_PinSocket_2.54mm:PinSocket_1x06_P2.54mm_Vertical, F.Cu at (158.1, 94.4)
Connections:
- net Net-(J2-Pad5) renamed /SCK
- net Net-(J2-Pad6) renamed /MISO
- net Net-(J2-Pad7) renamed /MOSI
- net Net-(J2-Pad8) renamed /CS
Routing:
- net +5V: track 229.3 -> 240.0 mm
- net /MISO: track 50.0 -> 43.3 mm
- net /SCK: track 55.2 -> 50.9 mm
- net /MOSI: track 44.3 -> 47.8 mm
- net /CS: track 51.7 -> 53.8 mm
Other:
- board text added: "+5V"
- board text added: "CLK"
- board text added: "CMD"
- board text added: "CS"
- board text added: "DAT"
- board text added: "MISO"
- board text added: "MOSI"
- board text added: "MZ-80K SD-CARD UNIT Rev1.5.3"
- board text added: "MicroSD Card Adapter"
- board text added: "SCK"
- board text added: "~CS"
- board text removed: "MZ-80K SD-CARD UNIT Rev1.5.2"

Commit message: Add files via upload
Parts:
- added R1: 10k, Resistor_THT:R_Axial_DIN0207_L6.3mm_D2.5mm_P7.62mm_Horizontal, F.Cu at (177.8, 94.0)
- added S3: 80K/700, Connector_PinHeader_2.54mm:PinHeader_1x03_P2.54mm_Vertical, F.Cu at (142.7, 58.9)
- moved C6 9.39 mm to (124.8, 68.8)
- moved S2 6.50 mm to (131.9, 59.1)
- moved S1 3.50 mm to (121.0, 59.1)
Connections:
- U2 pad 20: Net-(U2-Pad20) -> Net-(R1-Pad2)
- U5 pad 8: Net-(U2-Pad20) -> Net-(S3-Pad1)
Routing:
- net Net-(R1-Pad2): track 0.00 -> 112.4 mm
- net Net-(S3-Pad1): track 0.00 -> 75.5 mm, vias 0 -> 1
- net /D1: track 178.9 -> 139.2 mm, vias 1 -> 0
- net /D2: track 168.6 -> 134.4 mm, vias 1 -> 0
- net /A5: track 75.6 -> 104.0 mm, vias 1 -> 0
- net Net-(U2-Pad20): track 21.3 -> 0.00 mm
- net /A7: track 99.5 -> 119.7 mm, vias 1 -> 0
- net +5V: track 240.0 -> 257.1 mm
- net /A12: track 46.9 -> 34.3 mm, vias 0 -> 1
- net /D4: track 123.1 -> 112.7 mm, vias 1 -> 0
- net /A14: track 54.0 -> 44.3 mm, vias 0 -> 1
- net /A13: track 50.4 -> 40.9 mm, vias 0 -> 1
- net GND: track 352.8 -> 343.6 mm
- net /A4: track 88.3 -> 97.6 mm
- net /A15: track 57.7 -> 48.5 mm, vias 0 -> 1
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Other:
- board text added: "10k"
- board text added: "80K/700"
- board text added: "MZ-80K SD-CARD UNIT Rev1.5.5"
- board text removed: "MZ-80K SD-CARD UNIT Rev1.5.3"
