File: KiCad/MZ80k_SD/MZ80k_SD.sch (KiCad schematic (older format))
At the start: 13 parts, among them J1 MZ-80K BUS, J2 Micro_SD_Card_Kit, J3 INT VCC, J4 EXT 5V, U1 GAL22V10, U2 28C64, U3 8255, U4 Arduino_Pro_Mini_5V

Commit message: Add files via upload
Parts:
- added C4: 10uF, Capacitor_THT:CP_Radial_D5.0mm_P2.50mm, symbol Device:CP1
Connections:
- net +5V: now also C4.1
- net GND: now also C4.2
Changed lines of the file:
@@
 	800  4300 800  4500
 Connection ~ 800  4500
+$Comp
+L Device:CP1 C4
+U 1 1 61AFFCD6
+P 10450 3050
+F 0 "C4" H 10565 3096 50  0000 L CNN
+F 1 "10uF" H 10565 3005 50  0000 L CNN
+F 2 "Capacitor_THT:CP_Radial_D5.0mm_P2.50mm" H 10450 3050 50  0001 C CNN
+F 3 "~" H 10450 3050 50  0001 C CNN
+	1    10450 3050
+	1    0    0    -1
+$EndComp
+$Comp
+L power:GND #PWR013
+U 1 1 61B04D1B
+P 10450 3200
+F 0 "#PWR013" H 10450 2950 50  0001 C CNN
+F 1 "GND" H 10455 3027 50  0000 C CNN
+F 2 "" H 10450 3200 50  0001 C CNN
+F 3 "" H 10450 3200 50  0001 C CNN
+	1    10450 3200
+	1    0    0    -1
+$EndComp
 $EndSCHEMATC

Commit message: Add files via upload
Connections:
- net +5V: now also U2.1 (VPP)
- no-connect marks 47 -> 46
Changed lines of the file:
@@
 Wire Wire Line
 	5300 5100 5500 5100
-$Comp
-L Memory_EPROM:27C64 U2
-U 1 1 61A4CF3B
-P 6200 2600
-F 0 "U2" H 6000 3550 50  0000 C CNN
-F 1 "28C64" H 6400 3550 50  0000 C CNN
-F 2 "Package_DIP:DIP-28_W15.24mm_LongPads" H 6200 2600 50  0001 C CNN
-F 3 "http://ww1.microchip.com/downloads/en/DeviceDoc/11107M.pdf" H 6200 2600 50  0001 C CNN
-	1    6200 2600
-	1    0    0    -1
-$EndComp
 Wire Wire Line
 	5300 5500 5600 5500
@@
 Connection ~ 6200 3750
 Wire Wire Line
-	5700 3750 5700 3200
+	5700 3750 5700 3300
 Wire Wire Line
 	5700 1600 6200 1600
-Connection ~ 6200 1600
 $Comp
 L Device:C C3
@@
 Wire Wire Line
 	5700 3200 5700 1600
-NoConn ~ 5800 3300
 $Comp
 L power:GND #PWR04
@@
 	1    0    0    -1
 $EndComp
+Connection ~ 6200 1600
+$Comp
+L Memory_EPROM:27C64 U2
+U 1 1 61A4CF3B
+P 6200 2600
+F 0 "U2" H 6000 3550 50  0000 C CNN
+F 1 "28C64" H 6400 3550 50  0000 C CNN
+F 2 "Package_DIP:DIP-28_W15.24mm_LongPads" H 6200 2600 50  0001 C CNN
+F 3 "http://ww1.microchip.com/downloads/en/DeviceDoc/11107M.pdf" H 6200 2600 50  0001 C CNN
+	1    6200 2600
+	1    0    0    -1
+$EndComp
+Wire Wire Line
+	5800 3300 5700 3300
+Connection ~ 5700 3300
+Wire Wire Line
+	5700 3300 5700 3200
 $EndSCHEMATC

Commit message: Add files via upload
Parts:
- removed U1: GAL22V10, Package_DIP:DIP-24_W7.62mm_LongPads, symbol Memory_RAM2:GAL22V10
- added C4, C5: 0.1uF, Capacitor_THT:C_Rect_L4.0mm_W2.5mm_P2.50mm, symbol Device:C
- added U1: 74LS04, Package_DIP:DIP-14_W7.62mm_LongPads, symbol 74xx:74LS04
- added U5, U6: 74LS30, Package_DIP:DIP-14_W7.62mm_LongPads, symbol 74xx:74LS30
- C6: renamed from C4; value 10uF -> 100uF
- U2: value 28C64 -> 2764
Connections:
- net +5V: now also C1.2, C4.2, C5.2, U1.14 (VCC), U5.11, U5.12, U5.14 (VCC), U5.6, U6.12, U6.14 (VCC); no longer C1.1
- net GND: now also C1.1, J1.10 (Pin_10), J1.14 (Pin_14), J1.18 (Pin_18), J1.26 (Pin_26), J1.36 (Pin_36), J1.38 (Pin_38), J1.40 (Pin_40), J1.42 (Pin_42), J1.44 (Pin_44), J1.46 (Pin_46), J1.48 (Pin_48), J1.50 (Pin_50), J1.6 (Pin_6), C4.1, C5.1, U1.3, U1.5, U1.7 (GND), U5.7 (GND), U6.7 (GND); no longer C1.2
- net at U3.36 (~WR~): now also J1.20 (Pin_20)
- net at U3.5 (~RD~): now also J1.16 (Pin_16), U2.22 (~OE)
- net at U3.6 (~CS~): now also U6.8
- net at J1.1 (Pin_1): now also U5.1
- net at J1.27 (Pin_27), U2.8 (A2): now also U1.9
- net at J1.8 (Pin_8): now also U1.1
- net at J1.12 (Pin_12): now also U1.13
- net at J1.3 (Pin_3): now also U5.2
- net at U2.20 (~CE): now also U5.8
- net at J1.5 (Pin_5): now also U5.3
- net at J1.7 (Pin_7): now also U5.4
- net at J1.17 (Pin_17), U2.3 (A7): now also U6.6
- net at J1.19 (Pin_19), U2.4 (A6): now also U6.5
- net at J1.21 (Pin_21), U2.5 (A5): now also U1.11
- net at J1.23 (Pin_23), U2.6 (A4): now also U6.3
- net at J1.25 (Pin_25), U2.7 (A3): now also U6.2
- new net: U1.2, U5.5
- new net: U1.8, U6.1
- new net: U1.12, U6.11
- new net: U1.10, U6.4
- no-connect marks 46 -> 31
Other:
- moved on the sheet: C2, C3, C6, J2, J3, J4, S1, S2, U2, U3, U4

Commit message: Add files via upload
Connections:
- net GND: no longer U1.5
- net at J1.32 (Pin_32), U3.35 (RESET): now also U1.5
- net at U4.3 (RST): now also U1.6
- no-connect marks 31 -> 29
Other:
- moved on the sheet: U1C
Changed lines of the file:
@@
 Title "MZ-80K_SD"
 Date "2022-01-14"
-Rev "Rev1.5.1"
+Rev "Rev1.5.2"
 Comp ""
 Comment1 ""
@@
 NoConn ~ 10550 5600
 NoConn ~ 10050 4400
-NoConn ~ 10050 4300
 NoConn ~ 10050 4200
 NoConn ~ 10050 4100
@@
 L 74xx:74LS04 U1
 U 3 1 6232C3F4
-P 3750 8350
-F 0 "U1" H 3400 8500 50  0000 C CNN
-F 1 "74LS04" H 3950 8500 50  0000 C CNN
-F 2 "Package_DIP:DIP-14_W7.62mm_LongPads" H 3750 8350 50  0001 C CNN
-F 3 "http://www.ti.com/lit/gpn/sn74LS04" H 3750 8350 50  0001 C CNN
-	3    3750 8350
+P 8900 2900
+F 0 "U1" H 8550 3050 50  0000 C CNN
+F 1 "74LS04" H 9100 3050 50  0000 C CNN
+F 2 "Package_DIP:DIP-14_W7.62mm_LongPads" H 8900 2900 50  0001 C CNN
+F 3 "http://www.ti.com/lit/gpn/sn74LS04" H 8900 2900 50  0001 C CNN
+	3    8900 2900
 	1    0    0    -1
 $EndComp
@@
 Wire Wire Line
 	3450 7850 3300 7850
-Wire Wire Line
-	3300 7850 3300 8350
-Wire Wire Line
-	3300 8350 3450 8350
 $Comp
 L power:GND #PWR02
@@
 	1    0    0    -1
 $EndComp
-Wire Wire Line
-	3300 8450 3300 8350
-Connection ~ 3300 8350
 $Comp
 L Device:C C1
@@
 Connection ~ 5250 8700
 NoConn ~ 4050 7850
-NoConn ~ 4050 8350
 Wire Wire Line
 	9550 5200 10050 5200
@@
 Wire Wire Line
 	9550 6100 11600 6100
+Wire Wire Line
+	7950 3600 7950 2900
+Wire Wire Line
+	9950 2900 9950 4300
+Wire Wire Line
+	9950 4300 10050 4300
+Connection ~ 7950 3600
+Wire Wire Line
+	3300 7850 3300 8450
+Wire Wire Line
+	7950 2900 8600 2900
+Wire Wire Line
+	9200 2900 9950 2900
 $EndSCHEMATC

Commit message: Add files via upload
Connections:
- net D7: now reaches J1.35 (Pin_35), U2.19 (D7), U3.27 (D7)
- net D6: now reaches J1.37 (Pin_37), U2.18 (D6), U3.28 (D6)
- net D5: now reaches J1.39 (Pin_39), U2.17 (D5), U3.29 (D5)
- net D4: now reaches J1.41 (Pin_41), U2.16 (D4), U3.30 (D4)
- net D3: now reaches J1.43 (Pin_43), U2.15 (D3), U3.31 (D3)
- net D2: now reaches J1.45 (Pin_45), U2.13 (D2), U3.32 (D2)
- net D1: now reaches J1.47 (Pin_47), U2.12 (D1), U3.33 (D1)
- net D0: now reaches J1.49 (Pin_49), U2.11 (D0), U3.34 (D0)
- net RESET: now reaches J1.32 (Pin_32), U1.5, U3.35 (RESET)
- net ~WR: now reaches J1.20 (Pin_20), U3.36 (~WR~)
- net ~RD: now reaches J1.16 (Pin_16), U2.22 (~OE), U3.5 (~RD~)
- net A1: now reaches J1.29 (Pin_29), U2.9 (A1), U3.8 (A1)
- net A0: now reaches J1.31 (Pin_31), U2.10 (A0), U3.9 (A0)
- net A10: now reaches J1.11 (Pin_11), U2.21 (A10)
- net A11: now reaches J1.9 (Pin_9), U2.23 (A11)
- net A9: now reaches J1.13 (Pin_13), U2.24 (A9)
- net A8: now reaches J1.15 (Pin_15), U2.25 (A8)
- net A7: now reaches J1.17 (Pin_17), U2.3 (A7), U6.6
- net A6: now reaches J1.19 (Pin_19), U2.4 (A6), U6.5
- net A5: now reaches J1.21 (Pin_21), U1.11, U2.5 (A5)
- net A4: now reaches J1.23 (Pin_23), U2.6 (A4), U6.3
- net A3: now reaches J1.25 (Pin_25), U2.7 (A3), U6.2
- net A2: now reaches J1.27 (Pin_27), U1.9, U2.8 (A2)
- net A15: now reaches J1.1 (Pin_1), U5.1
- net ~IORQ: now reaches J1.12 (Pin_12), U1.13
- net A14: now reaches J1.3 (Pin_3), U5.2
- net A13: now reaches J1.5 (Pin_5), U5.3
- net A12: now reaches J1.7 (Pin_7), U5.4
- net ~MREQ: now reaches J1.8 (Pin_8), U1.1
Changed lines of the file:
@@
 Wire Wire Line
 	9200 2900 9950 2900
+Text Label 2100 5300 0    50   ~ 0
+D0
+Text Label 2100 5200 0    50   ~ 0
+D1
+Text Label 2100 5100 0    50   ~ 0
+D2
+Text Label 2100 5000 0    50   ~ 0
+D3
+Text Label 2100 4900 0    50   ~ 0
+D4
+Text Label 2100 4800 0    50   ~ 0
+D5
+Text Label 2100 4700 0    50   ~ 0
+D6
+Text Label 2100 4600 0    50   ~ 0
+D7
+Text Label 2100 4400 0    50   ~ 0
+A0
+Text Label 2100 4300 0    50   ~ 0
+A1
+Text Label 2100 4200 0    50   ~ 0
+A2
+Text Label 2100 4100 0    50   ~ 0
+A3
+Text Label 2100 4000 0    50   ~ 0
+A4
+Text Label 2100 3900 0    50   ~ 0
+A5
+Text Label 2100 3800 0    50   ~ 0
+A6
+Text Label 2100 3700 0    50   ~ 0
+A7
+Text Label 2100 3600 0    50   ~ 0
+A8
+Text Label 2100 3500 0    50   ~ 0
+A9
+Text Label 2100 3400 0    50   ~ 0
+A10
+Text Label 2100 3300 0    50   ~ 0
+A11
+Text Label 2100 3200 0    50   ~ 0
+A12
+Text Label 2100 3100 0    50   ~ 0
+A13
+Text Label 2100 3000 0    50   ~ 0
+A14
+Text Label 2100 2900 0    50   ~ 0
+A15
+Text Label 1450 3100 0    50   ~ 0
+GND
+Text Label 1400 3200 0    50   ~ 0
+~MREQ
+Text Label 1450 3300 0    50   ~ 0
+GND
+Text Label 1450 3500 0    50   ~ 0
+GND
+Text Label 1450 3700 0    50   ~ 0
+GND
+Text Label 1450 4100 0    50   ~ 0
+GND
+Text Label 1450 4500 0    50   ~ 0
+GND
+Text Label 1450 4600 0    50   ~ 0
+GND
+Text Label 1450 4700 0    50   ~ 0
+GND
+Text Label 1450 4800 0    50   ~ 0
+GND
+Text Label 1450 4900 0    50   ~ 0
+GND
+Text Label 1450 5000 0    50   ~ 0
+GND
+Text Label 1450 5100 0    50   ~ 0
+GND
+Text Label 1450 5200 0    50   ~ 0
+GND
+Text Label 1450 5300 0    50   ~ 0
+GND
+Text Label 1400 3400 0    50   ~ 0
+~IORQ
+Text Label 1500 3600 0    50   ~ 0
+~RD
+Text Label 1500 3800 0    50   ~ 0
+~WR
+Text Label 1400 4400 0    50   ~ 0
+RESET
 $EndSCHEMATC

Commit message: Add files via upload
Parts:
- added J5: MicroSD Card Adapter, Connector_PinSocket_2.54mm:PinSocket_1x06_P2.54mm_Vertical, symbol Connector_Generic:Conn_01x06
Connections:
- net +5V: now also J5.2 (Pin_2)
- net GND: now also J5.1 (Pin_1)
- net SCK: now reaches J2.5 (CLK), U4.16 (D13)
- net SCK: now also J5.5 (Pin_5)
- net MISO: now reaches J2.6 (DAT), U4.15 (D12)
- net MISO: now also J5.3 (Pin_3)
- net MOSI: now reaches J2.7 (CMD), U4.14 (~~D11)
- net MOSI: now also J5.4 (Pin_4)
- net CS: now reaches J2.8 (CS), U4.13 (~~D10)
- net CS: now also J5.6 (Pin_6)
Changed lines of the file:
@@
 Title "MZ-80K_SD"
 Date "2022-01-14"
-Rev "Rev1.5.2"
+Rev "Rev1.5.3"
 Comp ""
 Comment1 ""
@@
 Text Label 1400 4400 0    50   ~ 0
 RESET
+$Comp
+L Connector_Generic:Conn_01x06 J5
+U 1 1 62D11F48
+P 13050 3250
+F 0 "J5" H 13130 3242 50  0000 L CNN
+F 1 "MicroSD Card Adapter" H 12450 2800 50  0000 L CNN
+F 2 "Connector_PinSocket_2.54mm:PinSocket_1x06_P2.54mm_Vertical" H 13050 3250 50  0001 C CNN
+F 3 "~" H 13050 3250 50  0001 C CNN
+	1    13050 3250
+	1    0    0    -1
+$EndComp
+Wire Wire Line
+	12850 3050 12600 3050
+Wire Wire Line
+	12850 3150 12600 3150
+Wire Wire Line
+	12850 3250 12600 3250
+Wire Wire Line
+	12850 3350 12600 3350
+Wire Wire Line
+	12850 3450 12600 3450
+Wire Wire Line
+	12850 3550 12600 3550
+Text Label 11000 2200 0    50   ~ 0
+SCK
+Text Label 11000 2300 0    50   ~ 0
+MISO
+Text Label 11000 2400 0    50   ~ 0
+MOSI
+Text Label 11100 2500 0    50   ~ 0
+CS
+Text Label 12600 3050 0    50   ~ 0
+GND
+Text Label 12600 3150 0    50   ~ 0
++5V
+Text Label 12600 3250 0    50   ~ 0
+MISO
+Text Label 12600 3350 0    50   ~ 0
+MOSI
+Text Label 12600 3450 0    50   ~ 0
+SCK
+Text Label 12600 3550 0    50   ~ 0
+CS
 $EndSCHEMATC

Commit message: Add files via upload
Parts:
- added R1: 10k, Resistor_THT:R_Axial_DIN0207_L6.3mm_D2.5mm_P7.62mm_Horizontal, symbol Device:R
- added S3: 80K/700, Connector_PinHeader_2.54mm:PinHeader_1x03_P2.54mm_Vertical, symbol Memory_RAM2:SLIDE_SWITCH_3P
Connections:
- net +5V: now also R1.1
- net at U2.20 (~CE): now also R1.2, S3.2; no longer U5.8
- new net: S3.1, U5.8
- no-connect marks 29 -> 30
Changed lines of the file:
@@
 Title "MZ-80K_SD"
 Date "2022-01-14"
-Rev "Rev1.5.3"
+Rev "Rev1.5.5"
 Comp ""
 Comment1 ""
@@
 Connection ~ 6300 3200
 Wire Wire Line
-	6300 3200 6300 1600
+	6300 3200 6300 3100
 $Comp
 L power:GND #PWR04
@@
 Wire Wire Line
 	5500 4900 6100 4900
-Wire Wire Line
-	6100 4900 6100 3400
 $Comp
 L 74xx:74LS30 U6
@@
 Text Label 12600 3550 0    50   ~ 0
 CS
+$Comp
+L Memory_RAM2:SLIDE_SWITCH_3P S3
+U 1 1 66BA1EE1
+P 6300 4700
+F 0 "S3" H 6150 4650 50  0000 C CNN
+F 1 "80K/700" H 6500 4650 50  0000 C CNN
+F 2 "Connector_PinHeader_2.54mm:PinHeader_1x03_P2.54mm_Vertical" H 6300 4725 50  0001 C CNN
+F 3 "" H 6300 4725 50  0001 C CNN
+	1    6300 4700
+	1    0    0    -1
+$EndComp
+Wire Wire Line
+	6100 3400 6100 4200
+Wire Wire Line
+	6100 4200 6750 4200
+Wire Wire Line
+	6750 4200 6750 5200
+Wire Wire Line
+	6750 5200 6300 5200
+Wire Wire Line
+	6300 5200 6300 5050
+$Comp
+L Device:R R1
+U 1 1 66BE3A29
+P 6100 3250
+F 0 "R1" H 5900 3350 50  0000 L CNN
+F 1 "10k" H 5900 3200 50  0000 L CNN
+F 2 "Resistor_THT:R_Axial_DIN0207_L6.3mm_D2.5mm_P7.62mm_Horizontal" V 6030 3250 50  0001 C CNN
+F 3 "~" H 6100 3250 50  0001 C CNN
+	1    6100 3250
+	1    0    0    -1
+$EndComp
+Connection ~ 6100 3400
+Wire Wire Line
+	6100 3100 6300 3100
+Connection ~ 6300 3100
+Wire Wire Line
+	6300 3100 6300 1600
+NoConn ~ 6500 4900
 $EndSCHEMATC
